File: quadBLDC.sch (KiCad schematic (older format))
At the start: 0 parts

Commit message: Update: 回路図完成
Parts:
- added H1, H2, H3, H4: MountingHole, MountingHole:MountingHole_3.2mm_M3, symbol Mechanical:MountingHole
- added J1: CAN_CONN, Connector_JST:JST_PH_B4B-PH-K_1x04_P2.00mm_Vertical, symbol Connector_Generic:Conn_01x04
- added J10: VOUT_D, Connector_Wire:SolderWire-2.5sqmm_1x01_D2.4mm_OD3.6mm, symbol Connector_Generic:Conn_01x01
- added J11: GND, Connector_Wire:SolderWire-2.5sqmm_1x01_D2.4mm_OD3.6mm, symbol Connector_Generic:Conn_01x01
- added J2: RS422_CONN, Connector_JST:JST_PH_B4B-PH-K_1x04_P2.00mm_Vertical, symbol Connector_Generic:Conn_01x04
- added J3: SPI, Connector_JST:JST_PH_B6B-PH-K_1x06_P2.00mm_Vertical, symbol Connector_Generic:Conn_01x06
- added J4: VDC, Connector_Wire:SolderWire-2.5sqmm_1x01_D2.4mm_OD3.6mm, symbol Connector_Generic:Conn_01x01
- added J5: SWD, Connector_PinHeader_1.27mm:PinHeader_2x07_P1.27mm_Vertical_SMD, symbol Connector_Generic:Conn_02x07_Odd_Even
- added J6: Encoder, Connector_JST:JST_PHD_B8B-PHDSS_2x04_P2.00mm_Vertical, symbol Connector_Generic:Conn_02x04_Odd_Even
- added J7: VOUT_A, Connector_Wire:SolderWire-2.5sqmm_1x01_D2.4mm_OD3.6mm, symbol Connector_Generic:Conn_01x01
- added J8: VOUT_B, Connector_Wire:SolderWire-2.5sqmm_1x01_D2.4mm_OD3.6mm, symbol Connector_Generic:Conn_01x01
- added J9: VOUT_C, Connector_Wire:SolderWire-2.5sqmm_1x01_D2.4mm_OD3.6mm, symbol Connector_Generic:Conn_01x01
Connections:
- new net +3V3: J3.1 (Pin_1), J5.3 (Pin_3)
- new net +5V: J2.1 (Pin_1), J6.1 (Pin_1)
- new net +5VD: J1.1 (Pin_1)
- new net CAN_H: J1.3 (Pin_3)
- new net CAN_L: J1.4 (Pin_4)
- new net ENC_A+: J6.3 (Pin_3)
- new net ENC_A-: J6.4 (Pin_4)
- new net ENC_B+: J6.5 (Pin_5)
- new net ENC_B-: J6.6 (Pin_6)
- new net ENC_Z+: J6.7 (Pin_7)
- new net ENC_Z-: J6.8 (Pin_8)
- new net GND: J11.1 (Pin_1), J2.2 (Pin_2), J3.2 (Pin_2), J5.11 (Pin_11), J5.5 (Pin_5), J5.7 (Pin_7), J6.2 (Pin_2)
- new net GNDD: J1.2 (Pin_2)
- new net Inverter/VOUT_A: J7.1 (Pin_1)
- new net Inverter/VOUT_B: J8.1 (Pin_1)
- new net Inverter/VOUT_C: J9.1 (Pin_1)
- new net Inverter/VOUT_D: J10.1 (Pin_1)
- new net RS485_A: J2.3 (Pin_3)
- new net RS485_B: J2.4 (Pin_4)
- new net SPI_MISO: J3.5 (Pin_5)
- new net SPI_MOSI: J3.6 (Pin_6)
- new net SPI_NSS: J3.3 (Pin_3)
- new net SPI_SCK: J3.4 (Pin_4)
- new net T_NRST: J5.12 (Pin_12)
- new net T_SWCLK: J5.6 (Pin_6)
- new net T_SWDIO: J5.4 (Pin_4)
- new net T_SWO: J5.8 (Pin_8)
- new net T_VCP_RX: J5.13 (Pin_13)
- new net T_VCP_TX: J5.14 (Pin_14)
- new net VDC: J4.1 (Pin_1)
- no-connect marks 0 -> 4
