File: quadBLDC.sch (KiCad schematic (older format))
At the start: 15 parts, among them J1 CAN_CONN, J10 VOUT_D, J11 GND, J2 RS422_CONN, J3 SPI, J4 VDC, J5 SWD, J6 Encoder, J7 VOUT_A, J8 VOUT_B, J9 VOUT_C

Commit message: Update: 回路図、DCリンクCap1つ削除、アノテーションリセット
Parts:
- renumbered J9 to J10, J10 to J11, J5 to J4, J6 to J5, J4 to J6, J11 to J7, J7 to J8, J8 to J9
Changed lines of the file:
@@
 $EndSheet
 $Comp
-L power:GND #PWR011
+L power:GND #PWR012
 U 1 1 60D4AB1B
 P 13000 3600
-AR Path="/60D4AB1B" Ref="#PWR011"  Part="1"
+AR Path="/60D4AB1B" Ref="#PWR012"  Part="1"
 AR Path="/6093BF63/60D4AB1B" Ref="#PWR?"  Part="1"
-F 0 "#PWR011" H 13000 3350 50  0001 C CNN
+F 0 "#PWR012" H 13000 3350 50  0001 C CNN
 F 1 "GND" H 13005 3427 50  0000 C CNN
 F 2 "" H 13000 3600 50  0001 C CNN
@@
 $EndComp
 $Comp
-L power:VDC #PWR010
+L power:VDC #PWR011
 U 1 1 60D4AB24
 P 13000 2900
-AR Path="/60D4AB24" Ref="#PWR010"  Part="1"
+AR Path="/60D4AB24" Ref="#PWR011"  Part="1"
 AR Path="/6093BF63/60D4AB24" Ref="#PWR?"  Part="1"
-F 0 "#PWR010" H 13000 2800 50  0001 C CNN
+F 0 "#PWR011" H 13000 2800 50  0001 C CNN
 F 1 "VDC" H 13015 3073 50  0000 C CNN
 F 2 "" H 13000 2900 50  0001 C CNN
@@
 	13000 3500 13300 3500
 $Comp
-L Connector_Generic:Conn_02x07_Odd_Even J5
+L Connector_Generic:Conn_02x07_Odd_Even J4
 U 1 1 61CFD037
 P 3800 3650
-AR Path="/61CFD037" Ref="J5"  Part="1"
+AR Path="/61CFD037" Ref="J4"  Part="1"
 AR Path="/607D8C01/61CFD037" Ref="J?"  Part="1"
-F 0 "J5" H 3850 4167 50  0000 C CNN
+F 0 "J4" H 3850 4167 50  0000 C CNN
 F 1 "SWD" H 3850 4076 50  0000 C CNN
 F 2 "Connector_PinHeader_1.27mm:PinHeader_2x07_P1.27mm_Vertical_SMD" H 3800 3650 50  0001 C CNN
@@
 $EndComp
 $Comp
-L Connector_Generic:Conn_02x04_Odd_Even J6
+L Connector_Generic:Conn_02x04_Odd_Even J5
 U 1 1 61D0E831
 P 3900 8150
-F 0 "J6" H 3950 8467 50  0000 C CNN
+F 0 "J5" H 3950 8467 50  0000 C CNN
 F 1 "Encoder" H 3950 8376 50  0000 C CNN
 F 2 "Connector_JST:JST_PHD_B8B-PHDSS_2x04_P2.00mm_Vertical" H 3900 8150 50  0001 C CNN
@@
 	4250 8050 4250 8400
 $Comp
-L power:GND #PWR012
+L power:GND #PWR010
 U 1 1 61D2A888
 P 4250 8400
-AR Path="/61D2A888" Ref="#PWR012"  Part="1"
+AR Path="/61D2A888" Ref="#PWR010"  Part="1"
 AR Path="/607D8C01/61D2A888" Ref="#PWR?"  Part="1"
-F 0 "#PWR012" H 4250 8150 50  0001 C CNN
+F 0 "#PWR010" H 4250 8150 50  0001 C CNN
 F 1 "GND" H 4255 8227 50  0000 C CNN
 F 2 "" H 4250 8400 50  0001 C CNN
@@
 $EndComp
 $Comp
-L Connector_Generic:Conn_01x01 J7
+L Connector_Generic:Conn_01x01 J8
 U 1 1 63815069
 P 13500 4450
-F 0 "J7" H 13580 4492 50  0000 L CNN
+F 0 "J8" H 13580 4492 50  0000 L CNN
 F 1 "VOUT_A" H 13580 4401 50  0000 L CNN
 F 2 "Connector_Wire:SolderWire-2.5sqmm_1x01_D2.4mm_OD3.6mm" H 13500 4450 50  0001 C CNN
@@
 	11550 4650 13300 4650
 $Comp
-L Connector_Generic:Conn_01x01 J8
+L Connector_Generic:Conn_01x01 J9
 U 1 1 63818DC0
 P 13500 4650
-F 0 "J8" H 13580 4692 50  0000 L CNN
+F 0 "J9" H 13580 4692 50  0000 L CNN
 F 1 "VOUT_B" H 13580 4601 50  0000 L CNN
 F 2 "Connector_Wire:SolderWire-2.5sqmm_1x01_D2.4mm_OD3.6mm" H 13500 4650 50  0001 C CNN
@@
 	11550 4850 13300 4850
 $Comp
-L Connector_Generic:Conn_01x01 J9
+L Connector_Generic:Conn_01x01 J10
 U 1 1 6381BBB7
 P 13500 4850
-F 0 "J9" H 13580 4892 50  0000 L CNN
+F 0 "J10" H 13580 4892 50  0000 L CNN
 F 1 "VOUT_C" H 13580 4801 50  0000 L CNN
 F 2 "Connector_Wire:SolderWire-2.5sqmm_1x01_D2.4mm_OD3.6mm" H 13500 4850 50  0001 C CNN
@@
 	11550 5050 13300 5050
 $Comp
-L Connector_Generic:Conn_01x01 J10
+L Connector_Generic:Conn_01x01 J11
 U 1 1 6381EABC
 P 13500 5050
-F 0 "J10" H 13580 5092 50  0000 L CNN
+F 0 "J11" H 13580 5092 50  0000 L CNN
 F 1 "VOUT_D" H 13580 5001 50  0000 L CNN
 F 2 "Connector_Wire:SolderWire-2.5sqmm_1x01_D2.4mm_OD3.6mm" H 13500 5050 50  0001 C CNN
@@
 $EndComp
 $Comp
-L power:PWR_FLAG #FLG0101
+L power:PWR_FLAG #FLG04
 U 1 1 6394F0D8
 P 13000 3500
-F 0 "#FLG0101" H 13000 3575 50  0001 C CNN
+F 0 "#FLG04" H 13000 3575 50  0001 C CNN
 F 1 "PWR_FLAG" V 13000 3628 50  0000 L CNN
 F 2 "" H 13000 3500 50  0001 C CNN
@@
 	13000 3600 13000 3500
 $Comp
-L power:PWR_FLAG #FLG0102
+L power:PWR_FLAG #FLG03
 U 1 1 6394FE58
 P 13000 3000
-F 0 "#FLG0102" H 13000 3075 50  0001 C CNN
+F 0 "#FLG03" H 13000 3075 50  0001 C CNN
 F 1 "PWR_FLAG" V 13000 3127 50  0000 L CNN
 F 2 "" H 13000 3000 50  0001 C CNN
@@
 $EndComp
 $Comp
-L power:PWR_FLAG #FLG0103
+L power:PWR_FLAG #FLG01
 U 1 1 63951D45
 P 3550 5150
-F 0 "#FLG0103" H 3550 5225 50  0001 C CNN
+F 0 "#FLG01" H 3550 5225 50  0001 C CNN
 F 1 "PWR_FLAG" V 3550 5278 50  0000 L CNN
 F 2 "" H 3550 5150 50  0001 C CNN
@@
 	3550 5150 3550 5300
 $Comp
-L power:PWR_FLAG #FLG0104
+L power:PWR_FLAG #FLG02
 U 1 1 63957E09
 P 3550 5800
-F 0 "#FLG0104" H 3550 5875 50  0001 C CNN
+F 0 "#FLG02" H 3550 5875 50  0001 C CNN
 F 1 "PWR_FLAG" V 3550 5928 50  0000 L CNN
 F 2 "" H 3550 5800 50  0001 C CNN
@@
 	3550 5800 3550 5850
 $Comp
-L Connector_Generic:Conn_01x01 J4
+L Connector_Generic:Conn_01x01 J6
 U 1 1 6397F3DB
 P 13500 3000
-F 0 "J4" H 13580 3042 50  0000 L CNN
+F 0 "J6" H 13580 3042 50  0000 L CNN
 F 1 "VDC" H 13580 2951 50  0000 L CNN
 F 2 "Connector_Wire:SolderWire-2.5sqmm_1x01_D2.4mm_OD3.6mm" H 13500 3000 50  0001 C CNN
@@
 $EndComp
 $Comp
-L Connector_Generic:Conn_01x01 J11
+L Connector_Generic:Conn_01x01 J7
 U 1 1 6398B579
 P 13500 3500
-F 0 "J11" H 13580 3542 50  0000 L CNN
+F 0 "J7" H 13580 3542 50  0000 L CNN
 F 1 "GND" H 13580 3451 50  0000 L CNN
 F 2 "Connector_Wire:SolderWire-2.5sqmm_1x01_D2.4mm_OD3.6mm" H 13500 3500 50  0001 C CNN
