File: Inverter.sch (KiCad schematic (older format))
At the start: 96 parts, among them Q1 NTMFS5C670NL, Q2 NTMFS5C670NL, Q3 NTMFS5C670NL, Q4 NTMFS5C670NL, Q5 NTMFS5C670NL, Q6 NTMFS5C670NL, Q7 NTMFS5C670NL, Q8 NTMFS5C670NL, U1 LM5109BMA, U10 NJU77701F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

Commit message: Fix: ゲートドライブの配線修正
Connections:
- net VOUT_A: now also C4.2, U1.6 (HS)
- net VOUT_B: now also C11.2, U4.6 (HS)
- net VOUT_C: now also C18.2, U7.6 (HS)
- net VOUT_D: now also C24.2, U9.6 (HS)
Changed lines of the file:
@@
 	0    1    1    0
 $EndComp
+Wire Wire Line
+	3750 4000 4300 4000
+Wire Wire Line
+	4300 4000 4300 3700
+Wire Wire Line
+	4300 3700 4500 3700
+Connection ~ 3750 4000
+Wire Wire Line
+	6800 4000 7350 4000
+Wire Wire Line
+	7350 4000 7350 3700
+Wire Wire Line
+	7350 3700 7550 3700
+Wire Wire Line
+	9850 4000 10400 4000
+Wire Wire Line
+	10400 4000 10400 3700
+Wire Wire Line
+	10400 3700 10600 3700
+Wire Wire Line
+	12900 4000 13450 4000
+Wire Wire Line
+	13450 4000 13450 3700
+Wire Wire Line
+	13450 3700 13650 3700
+Connection ~ 12900 4000
+Connection ~ 9850 4000
+Connection ~ 6800 4000
 Wire Bus Line
 	11550 4000 11550 7450
