File: quadBLDC.kicad_pcb (KiCad board)
At the start: 2 copper layers, 100 x 100 mm, 163 parts, among them IC1 STM32G474RET6, J1 CAN_CONN, J10 VOUT_D, J11 GND, J2 RS422_CONN, J3 SPI, J4 VDC, J5 SWD, J6 Encoder, J7 VOUT_A, J8 VOUT_B, J9 VOUT_C, Q1 NTMFS5C670NL, Q2 NTMFS5C670NL, Q3 NTMFS5C670NL, Q4 NTMFS5C670NL, Q5 NTMFS5C670NL, Q6 NTMFS5C670NL, Q7 NTMFS5C670NL, Q8 NTMFS5C670NL, SW1 RST, SW2 SW_DIP_x04, U1 LM5109BMA, U10 NJU77701F, U11 MCP1825S, U12 MP2456GJ-Z, U13 TLV75533PDBV, U14 MCP2562-E-SN, U15 ST1480ABDR, U16 AM26LV32ACPWR, U17 SI8621AB-B-ISR, U2 NJU77701F, U3 NJU77701F, U4 LM5109BMA, U5 NJU77701F, U6 NJU77701F, U7 LM5109BMA, U8 NJU77701F, U9 LM5109BMA, Y1 Resonator_Small

Commit message: wip: レグの配置途中
Parts:
- C1, C4: moved to B.Cu
- moved H1 149.6 mm to (3.00, 3.00)
- moved J10 148.0 mm to (14.0, 4.00)
- moved R1 144.5 mm to (49.0, 72.5)
- moved Q8 137.8 mm to (11.0, 16.0), turned to 90 degrees
- moved C1 133.9 mm to (53.5, 72.5), turned to 180 degrees
- moved Q6 133.1 mm to (25.0, 16.0), turned to 90 degrees
- moved H2 131.0 mm to (3.00, 97.0)
- moved C5 129.6 mm to (51.5, 83.0), turned to 90 degrees
- moved J9 129.0 mm to (28.0, 4.00)
- moved R6 124.1 mm to (53.0, 83.0), turned to 90 degrees
- moved R5 119.9 mm to (56.0, 65.0), turned to 180 degrees
- moved C4 119.8 mm to (53.0, 67.5)
- moved C7 119.7 mm to (50.0, 62.5)
- moved NT2 117.9 mm to (72.0, 80.5), turned to 90 degrees
- moved J8 116.5 mm to (42.0, 4.00)
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
Commit message: wip: レグ配置中
Parts:
- moved C14 122.8 mm to (42.5, -39.5)
- moved R20 104.7 mm to (47.5, -42.0), turned to 270 degrees
- moved C1 102.1 mm to (57.5, -29.5)
- moved C4 102.1 mm to (57.0, -34.5)
- moved C7 102.1 mm to (54.0, -39.5)
- moved U1 102.1 mm to (57.5, -32.0)
- moved D1 102.1 mm to (52.0, -34.0)
- moved Q2 102.1 mm to (58.5, -50.0)
- moved R8 102.1 mm to (59.0, -42.0)
- moved R7 101.7 mm to (56.0, -36.6)
- moved C5 101.7 mm to (55.3, -18.6)
- moved C6 101.7 mm to (59.8, -12.6)
- moved NT1 101.7 mm to (77.3, -23.6)
- moved NT2 101.7 mm to (75.8, -21.1)
- moved R2 101.7 mm to (60.8, -22.1)
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Connections:
- C11 pad 2: Net-(C11-Pad2) -> /Inverter/VOUT_B
- C14 pad 2: Net-(C14-Pad2) -> GND
- C18 pad 2: Net-(C18-Pad2) -> /Inverter/VOUT_C
- C22 pad 2: Net-(C22-Pad2) -> GND
- C24 pad 2: Net-(C24-Pad2) -> /Inverter/VOUT_D
- C27 pad 2: Net-(C27-Pad2) -> GND
- C4 pad 2: Net-(C4-Pad2) -> /Inverter/VOUT_A
- C7 pad 2: Net-(C7-Pad2) -> GND
- NT1 pad 1: Net-(C7-Pad2) -> Net-(NT1-Pad1)
- NT3 pad 1: Net-(C14-Pad2) -> Net-(NT3-Pad1)
- NT5 pad 1: Net-(C22-Pad2) -> Net-(NT5-Pad1)
- NT7 pad 1: Net-(C27-Pad2) -> Net-(NT7-Pad1)
- Q2 pad 1: Net-(C7-Pad2) -> Net-(NT1-Pad1)
- Q2 pad 2: Net-(C7-Pad2) -> Net-(NT1-Pad1)
- Q2 pad 3: Net-(C7-Pad2) -> Net-(NT1-Pad1)
- Q4 pad 1: Net-(C14-Pad2) -> Net-(NT3-Pad1)
- Q4 pad 2: Net-(C14-Pad2) -> Net-(NT3-Pad1)
- Q4 pad 3: Net-(C14-Pad2) -> Net-(NT3-Pad1)
- Q6 pad 1: Net-(C22-Pad2) -> Net-(NT5-Pad1)
- Q6 pad 2: Net-(C22-Pad2) -> Net-(NT5-Pad1)
- Q6 pad 3: Net-(C22-Pad2) -> Net-(NT5-Pad1)
- Q8 pad 1: Net-(C27-Pad2) -> Net-(NT7-Pad1)
- Q8 pad 2: Net-(C27-Pad2) -> Net-(NT7-Pad1)
- Q8 pad 3: Net-(C27-Pad2) -> Net-(NT7-Pad1)
- R20 pad 1: Net-(C14-Pad2) -> Net-(NT3-Pad1)
- R31 pad 1: Net-(C22-Pad2) -> Net-(NT5-Pad1)
- R39 pad 1: Net-(C27-Pad2) -> Net-(NT7-Pad1)
- R8 pad 1: Net-(C7-Pad2) -> Net-(NT1-Pad1)
- U1 pad 6: Net-(C4-Pad2) -> /Inverter/VOUT_A
- U4 pad 6: Net-(C11-Pad2) -> /Inverter/VOUT_B
- U7 pad 6: Net-(C18-Pad2) -> /Inverter/VOUT_C
- U9 pad 6: Net-(C24-Pad2) -> /Inverter/VOUT_D

Commit message: wip: レグ配線中
Parts:
- added C50: 1uF/50V, Capacitor_SMD:C_0805_2012Metric, F.Cu at (55.0, 21.0)
- added C51: 1uF/50V, Capacitor_SMD:C_0805_2012Metric, F.Cu at (43.0, 21.0)
- added C52: 1uF/50V, Capacitor_SMD:C_0805_2012Metric, F.Cu at (31.0, 21.0)
- added C53: 1uF/50V, Capacitor_SMD:C_0805_2012Metric, F.Cu at (19.0, 21.0)
- C10, C11, C16, C18, C23, C24: moved to B.Cu
- moved C26 162.7 mm to (16.0, 44.5)
- moved R34 159.5 mm to (22.0, 50.5)
- moved R37 154.7 mm to (22.0, 53.5)
- moved C25 154.5 mm to (21.5, 55.5)
- moved U10 146.5 mm to (22.5, 42.0), turned to 180 degrees
- moved NT7 145.9 mm to (25.0, 16.5), turned to 270 degrees
- moved R36 140.1 mm to (25.5, 26.0), turned to 270 degrees
- moved U8 139.1 mm to (35.0, 42.0), turned to 180 degrees
- moved R32 138.6 mm to (19.0, 34.5)
- moved NT6 138.3 mm to (37.0, 20.5), turned to 90 degrees
- moved R38 138.2 mm to (23.5, 26.0), turned to 270 degrees
- moved R25 138.0 mm to (35.0, 52.5)
- moved R23 135.7 mm to (31.0, 34.5)
- moved R14 135.2 mm to (43.5, 42.5), turned to 180 degrees
- moved C19 135.1 mm to (35.5, 57.0)
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Routing:
- net /Inverter/VOUT_A: track 0.00 -> 41.8 mm, vias 0 -> 1
- net /Inverter/VOUT_D: track 0.00 -> 31.3 mm, vias 0 -> 1
- net /Inverter/VOUT_C: track 0.00 -> 31.3 mm, vias 0 -> 1
- net /Inverter/VOUT_B: track 0.00 -> 31.3 mm, vias 0 -> 1
- net Net-(Q8-Pad4): track 0.00 -> 22.5 mm, vias 0 -> 2
- net Net-(Q4-Pad4): track 0.00 -> 22.2 mm, vias 0 -> 2
- net Net-(Q2-Pad4): track 0.00 -> 22.2 mm, vias 0 -> 2
- net Net-(Q6-Pad4): track 0.00 -> 22.2 mm, vias 0 -> 2
- net Net-(NT1-Pad2): track 0.00 -> 20.2 mm
- net Net-(NT2-Pad2): track 0.00 -> 19.3 mm
- net Net-(Q1-Pad4): track 0.00 -> 18.6 mm
- net Net-(Q3-Pad4): track 0.00 -> 18.4 mm
- net Net-(Q7-Pad4): track 0.00 -> 18.4 mm
- net Net-(Q5-Pad4): track 0.00 -> 18.4 mm
- net Net-(NT5-Pad2): track 0.00 -> 13.7 mm
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- added copper zone on F.Cu, net /Inverter/VOUT_A
- added copper zone on F.Cu, net /Inverter/VOUT_B
- added copper zone on F.Cu, net /Inverter/VOUT_C
- added copper zone on F.Cu, net /Inverter/VOUT_D
- added copper zone on B.Cu, net GND
- added copper zone on F.Cu, net GND
- added copper zone on F.Cu, net Net-(NT1-Pad1)
- added copper zone on F.Cu, net Net-(NT3-Pad1)
- added copper zone on F.Cu, net Net-(NT5-Pad1)
- added copper zone on F.Cu, net Net-(NT7-Pad1)
- added copper zone on B.Cu, net VDC
- added copper zone on F.Cu, net VDC

Commit message: wip: 配置
Parts:
- moved C37 200.5 mm to (55.9, 139.2)
- moved C44 200.5 mm to (43.0, 141.0)
- moved C45 200.5 mm to (59.7, 124.1)
- moved C46 200.5 mm to (57.6, 126.7)
- moved C49 200.5 mm to (43.0, 138.5)
- moved D7 200.5 mm to (55.7, 121.6)
- moved R49 200.5 mm to (55.9, 134.2)
- moved R51 200.5 mm to (57.6, 131.7)
- moved C38 200.5 mm to (59.7, 121.6)
- moved C39 200.5 mm to (55.7, 124.1)
- moved C40 200.5 mm to (53.6, 128.0)
- moved C41 200.5 mm to (47.9, 132.5)
- moved C42 200.5 mm to (53.6, 130.5)
- moved C43 200.5 mm to (47.9, 135.1)
- moved C47 200.5 mm to (47.9, 137.6)
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Routing:
- net GND: track 6.54 -> 22.0 mm, vias 56 -> 60
- net +12V: track 10.1 -> 25.6 mm, vias 0 -> 4
- net Net-(NT4-Pad2): track 12.6 -> 19.2 mm
- net Net-(NT8-Pad2): track 12.6 -> 19.1 mm
- net Net-(NT6-Pad2): track 12.6 -> 19.1 mm
- net Net-(NT3-Pad2): track 13.7 -> 20.1 mm
- net Net-(NT5-Pad2): track 13.7 -> 20.0 mm
- net Net-(NT7-Pad2): track 13.7 -> 20.0 mm

Commit message: wip: 配置
Parts:
- moved R45 79.8 mm to (-18.0, 117.0)
- moved R52 72.5 mm to (63.5, 69.5)
- moved C40 71.6 mm to (-18.0, 126.5)
- moved SW1 71.1 mm to (69.0, 61.0)
- moved Y1 71.1 mm to (35.5, 64.5), turned to 270 degrees
- moved R50 69.7 mm to (75.5, 72.5)
- moved C44 63.0 mm to (51.0, 78.5)
- moved C41 62.5 mm to (-13.7, 122.0)
- moved SW2 60.7 mm to (8.50, 81.0)
- moved R46 60.5 mm to (-8.00, 154.0)
- moved C43 60.0 mm to (65.0, 77.5)
- moved C47 59.9 mm to (58.0, 78.5)
- moved NT9 59.2 mm to (47.0, 84.5)
- moved C38 59.0 mm to (2.50, 136.0)
- moved C42 56.1 mm to (38.5, 76.5)
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Routing:
- net GND: track 22.0 -> 41.9 mm, vias 60 -> 62
- net Net-(C32-Pad2): track 0.00 -> 11.5 mm
- net +12V: track 25.6 -> 34.9 mm
- net VDC: track 0.00 -> 8.48 mm
- net Net-(R41-Pad1): track 0.00 -> 6.04 mm
- net Net-(R40-Pad2): track 0.00 -> 3.53 mm
- net Net-(C32-Pad1): track 0.00 -> 2.18 mm
- net Net-(C34-Pad2): track 0.00 -> 1.93 mm

Commit message: wip: 配置
Parts:
- removed the C3 at (79.0, 12.5)
- moved C1 12.0 mm to (79.5, 12.5)
- renumbered C2 to C1, C9 to C10, C51 to C15, C15 to C17, C1 to C2, C17 to C20, C20 to C21, C21 to C22, C22 to C23, C52 to C24, C23 to C25, C24 to C26, C25 to C27, C26 to C28, C27 to C29, C4 to C3, C53 to C30, C28 to C31, C29 to C32, C30 to C33, C31 to C34, C32 to C35, C33 to C36, C34 to C37, C35 to C38, C36 to C39, C5 to C4, C37 to C40, C38 to C41, C39 to C42, C40 to C43, C41 to C44, C42 to C45, C43 to C46, C44 to C47, C45 to C48, C46 to C49, C6 to C5, C47 to C50, C48 to C51, C49 to C52, C7 to C6, C50 to C7, C10 to C8, C8 to C9, J9 to J10, J10 to J11, J5 to J4, J6 to J5, J4 to J6, J11 to J7, J7 to J8, J8 to J9, R13 to R12, R12 to R13, R30 to R29, R31 to R30, R29 to R31, U7 to U6, U6 to U7

Commit message: Update: アナログリファレンスをLDOからに変更
Parts:
- removed the C48 at (74.5, 78.5)
- removed the C49 at (56.0, 72.0)
- removed the C50 at (58.0, 78.5)
- removed FB1: Ferrite_Bead_Small, Inductor_SMD:L_0603_1608Metric
- added C37: 1uF/16V, Capacitor_SMD:C_0603_1608Metric, F.Cu at (149.0, -8.59)
- added C40: 1uF/16V, Capacitor_SMD:C_0603_1608Metric, F.Cu at (153.9, -13.2)
- added C42: 0.1uF/16V, Capacitor_SMD:C_0603_1608Metric, F.Cu at (153.0, -8.59)
- added C43: 0.01uF/16V, Capacitor_SMD:C_0603_1608Metric, F.Cu at (157.9, -13.2)
- added U14: TLV75533PDBV, Package_TO_SOT_SMD:SOT-23-5, F.Cu at (149.4, -12.2)
- moved NT9 142.9 mm to (153.4, -11.0)
- renumbered C37 to C38, C38 to C39, C39 to C41, C40 to C44, C41 to C45, C42 to C46, C43 to C47, C44 to C48, C45 to C49, C46 to C50, C47 to C51, C51 to C52, C52 to C53, U14 to U15, U15 to U16, U16 to U17, U17 to U18
Connections:
- net VDDA renamed +3.3VA

Commit message: wip
Parts:
- moved C43 82.7 mm to (95.0, 40.5), turned to 180 degrees
- moved C41 81.7 mm to (90.5, 36.5), turned to 180 degrees
- moved C36 80.9 mm to (90.5, 30.5), turned to 180 degrees
- moved U13 78.5 mm to (90.5, 33.5), turned to 270 degrees
- moved C40 77.1 mm to (95.0, 36.5), turned to 180 degrees
- moved C42 74.7 mm to (95.0, 38.5), turned to 180 degrees
- moved U14 71.1 mm to (95.0, 33.5), turned to 270 degrees
- moved C10 70.4 mm to (133.0, 24.0)
- moved C9 70.4 mm to (128.0, 21.0)
- moved R10 70.4 mm to (132.0, 17.5)
- moved R11 70.4 mm to (136.0, 21.0)
- moved R13 70.4 mm to (130.0, 21.0)
- moved R9 70.4 mm to (134.0, 17.5)
- moved U3 70.4 mm to (133.0, 21.0)
- moved NT9 69.4 mm to (96.0, 28.0), turned to 270 degrees
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