File: quadBLDC.kicad_pcb (KiCad board)
At the start: 2 copper layers, 100 x 100 mm, 423 parts, among them IC1 STM32G474RET6, J1 CAN_CONN, J10 VOUT_C, J11 VOUT_D, J2 RS422_CONN, J3 SPI, J4 SWD, J5 Encoder, J6 VDC, J7 GND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

Commit message: Add: ガーバー書き出し
Routing:
- net GND: vias 126 -> 125
Other:
- rule pad_to_mask_clearance: 0.05 -> 0
